File: KiCAD/MixtapeNEO-3000.kicad_pcb (KiCad board)
At the start: 2 copper layers, 99 x 64.8 mm, 52 parts, among them J1 CONN_01X04, J18 Con_3-5V, J2 CONN_01X04, J3 CONN_02X03, J5 CONN_01X02_MALE, J7 USB_OTG, SW1 SW_Push, SW2 SW_Push, SW3 SW_Push, SW6 SW_Push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

Commit message: all footprints done
Parts:
- removed J18: Con_3-5V, 8BitMixtape-3000:Bat_connector
- removed J7: USB_OTG, 8BitMixtape-3000:USB_Micro-B
- removed SW6: SW_Push, 8Bit-MOJ-MIKRO-Kaseta:SW_SPST_FSMSM
- added BT1: Battery_Cell, 8BitMixtape-3000:BAT_Holder_AAA-new, B.Cu at (149.3, 87.3)
- added BT2: Battery_Cell, 8BitMixtape-3000:BAT_Holder_AAA-new, B.Cu at (149.3, 123.5)
- added J4: Con_3-5V, 8BitMixtape-3000:Bat_connector, B.Cu at (109.7, 87.1)
- added J6: CONN_01X02_MALE, Resistors_SMD:R_0612, B.Cu at (157.5, 59.8)
- added SW4: SW_Push, 8BitMixtape-3000:SW_SPST_FSMSM, B.Cu at (166.2, 60.2)
- C5: value 1uF -> 10uF
- C6: value 10uF -> 1uF
- C7: value 10uF -> 220uF
- J5: value CONN_01X02_MALE -> USB_OTG; footprint Resistors_SMD:R_0612 -> 8BitMixtape-3000:USB_Micro-B
- POT1-MAIN1, POT2-CV1: footprint 8BitMixtape-3000:Poti_Mouser -> 8BitMixtape-3000:Potentiometer_backPads_noHole
- POT3-Vol1: footprint 8Bit_ESPTINY86-Mixtape:Potentiometer_wheel -> 8BitMixtape-3000:Potentiometer_wheel
- SW1: footprint 8Bit-MOJ-MIKRO-Kaseta:Push_SWITCH_hole -> 8BitMixtape-3000:Push_SWITCH_hole
- U3: moved to B.Cu
- moved U3 12.7 mm to (164.8, 51.8)
- moved R10 2.97 mm to (132.7, 123.2)
- moved POT1-MAIN1 2.67 mm to (175.7, 113.2)
- moved POT2-CV1 2.42 mm to (134.3, 113.4)
- moved C4 0.45 mm to (149.7, 122.5)
Connections:
- C5 pad 2: GND -> Sound_OUT
- C6 pad 2: Sound_OUT -> GND
- C7 pad 1: GND -> VCC
- C7 pad 2: VCC -> GND
- J5 pad 1: Net-(J5-Pad1) -> VCC
- J5 pad 2: Sync_OUT -> (no net)
- R14 pad 2: Net-(C6-Pad1) -> Net-(C5-Pad1)
- U1 pad 1: Net-(J5-Pad1) -> Net-(J6-Pad1)
- U2 pad 2: Net-(C5-Pad1) -> Net-(C6-Pad1)
- U2 pad 3: Net-(C5-Pad1) -> Net-(C6-Pad1)
