File: KiCAD/MixtapeNEO-3000.kicad_pcb (KiCad board)
At the start: 2 copper layers, 99 x 64.8 mm, 54 parts, among them J1 CONN_01X04, J2 CONN_01X04, J3 CONN_02X03, J4 Con_3-5V, J5 USB_OTG, J6 CONN_01X02_MALE, SW1 SW_Push, SW2 SW_Push, SW3 SW_Push, SW4 SW_Push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

Commit message: complete revision
Parts:
- removed J3: CONN_02X03, 8BitMixtape-3000:Socket_Strip_Straight_2x03_Pitch2.54mm
- removed J5: USB_OTG, 8BitMixtape-3000:USB_Micro-B
- removed SW4: SW_Push, 8BitMixtape-3000:SW_SPST_FSMSM
- removed U3: 7805, TO_SOT_Packages_SMD:TO-252-3_TabPin2
- added R99: 0, 8BitMixtape-3000-clean:R_1206_HandSoldering, F.Cu at (109.2, 83.8)
- BT1, BT2: footprint 8BitMixtape-3000:BAT_Holder_AAA-new -> 8BitMixtape-3000-clean:BAT_Holder_AAA-new_noHole
- C1, C2, C3, C4, C5, C6, C7: footprint 8BitMixtape-3000:C_1206_HandSoldering -> 8BitMixtape-3000-clean:C_1206_HandSoldering
- D-OUT1, D-POW1: footprint 8BitMixtape-3000:LED_2835_minimal -> 8BitMixtape-3000-clean:LED_2835_minimal
- J1, J2: footprint 8BitMixtape-3000:Angled_1x04_Pitch2.54mm-flip -> 8BitMixtape-3000-clean:Angled_1x04_Pitch2.54mm-flip
- J4: footprint 8BitMixtape-3000:Bat_connector -> 8BitMixtape-3000-clean:Bat_connector_SMD
- J6: footprint Resistors_SMD:R_0612 -> 8BitMixtape-3000-clean:R_0612
- Jack1, Jack2: footprint 8BitMixtape-3000:AUDIO-Jack_3.5mm_5Pin -> 8BitMixtape-3000-clean:AUDIO-Jack_3.5mm_5Pin
- NEO1, NEO2, NEO3, NEO4, NEO5, NEO6, NEO7, NEO8: footprint 8BitMixtape-3000:Mixtape_NEO_WS2812B -> 8BitMixtape-3000-clean:Mixtape_NEO_WS2812B
- POT1-MAIN1, POT2-CV1: footprint 8BitMixtape-3000:Potentiometer_backPads_noHole -> 8BitMixtape-3000-clean:Potentiometer_backPads_noHole
- POT3-Vol1: footprint 8BitMixtape-3000:Potentiometer_wheel -> 8BitMixtape-3000-clean:Potentiometer_wheel
- R1, R10, R11, R12, R13, R14, R15, R2, R3, R4, R5, R6, R7, R8, R9: footprint 8BitMixtape-3000:R_1206_HandSoldering -> 8BitMixtape-3000-clean:R_1206_HandSoldering
- SW1: footprint 8BitMixtape-3000:Push_SWITCH_hole -> 8BitMixtape-3000-clean:Push_SWITCH_hole
- SW2, SW3: footprint 8BitMixtape-3000:SW_PUSH-12mm_3D -> 8BitMixtape-3000-clean:TACTILE-PTH_6mm_SMD
- Speaker1: footprint 8BitMixtape-3000:Socket_Strip_Straight_1x02_Pitch2.54mm -> 8BitMixtape-3000-clean:SpeakerPads_SMD
- U1: footprint 8BitMixtape-3000:Attiny_DIP-8_W7.62mm -> 8BitMixtape-3000-clean:Attiny_DIP-8_W7.62mm_mod
- U2: footprint Housings_SOIC:SO-8_5.3x6.2mm_Pitch1.27mm -> 8BitMixtape-3000-clean:SO-8_5.3x6.2mm_Pitch1.27mm
- board1: footprint 8BitMixtape-3000:MixtapeNEO-3000 -> 8BitMixtape-3000-clean:MixtapeNEO-3000
- moved Speaker1 43.1 mm to (193.3, 118.4), turned to 270 degrees
- moved U2 43.0 mm to (188.9, 122.9)
- moved J6 42.6 mm to (142.5, 99.7)
- moved C6 41.5 mm to (186.2, 128.3)
- moved R15 41.1 mm to (189.0, 117.9), turned to 180 degrees
- moved C7 39.9 mm to (192.0, 128.3), turned to 180 degrees
- moved C2 38.6 mm to (149.8, 110.9), turned to 180 degrees
- moved R8 30.9 mm to (190.8, 84.1), turned to 0 degrees
- moved R11 24.8 mm to (157.7, 118.9)
- moved C5 24.2 mm to (186.7, 84.1), turned to 90 degrees
- moved R14 18.2 mm to (189.5, 84.1), turned to 90 degrees
- moved R3 15.9 mm to (146.7, 118.9), turned to 270 degrees
- moved R5 15.7 mm to (149.9, 118.9), turned to 270 degrees
- moved C3 14.6 mm to (190.8, 81.8), turned to 0 degrees
- moved R4 11.5 mm to (153.0, 118.9), turned to 270 degrees
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Connections:
- J2 pad 3: Sound_OUT -> PB1
- Jack1 pad 2: CV_IN -> Net-(Jack1-Pad2)
- Jack2 pad 2: Sound_OUT -> Net-(Jack2-Pad2)
- Jack2 pad 5: (no net) -> Sound_OUT
- POT2-CV1 pad 1: Sound_IN -> CV_IN
- POT3-Vol1 pad 2: Sound_OUT -> Net-(Jack2-Pad2)
- R10 pad 2: Sound_IN -> CV_IN
Routing:
- net VCC: track 0.00 -> 271.5 mm, vias 0 -> 9
- net GND: track 0.00 -> 169.0 mm, vias 0 -> 9
- net CV_IN: track 0.00 -> 94.5 mm, vias 0 -> 4
- net PB3: track 0.00 -> 89.2 mm, vias 0 -> 1
- net Sync_OUT: track 0.00 -> 88.0 mm
- net PB1: track 0.00 -> 82.0 mm
- net But-R: track 0.00 -> 43.2 mm
- net Net-(R14-Pad1): track 0.00 -> 40.3 mm, vias 0 -> 2
- net Net-(NEO1-Pad2): track 0.00 -> 39.2 mm, vias 0 -> 2
- net Net-(BT1-Pad2): track 0.00 -> 36.6 mm
- net But-L: track 0.00 -> 35.1 mm
- net Net-(POT1-MAIN1-Pad1): track 0.00 -> 26.1 mm, vias 0 -> 1
- net +3V3: track 0.00 -> 23.0 mm
- net Net-(Jack2-Pad2): track 0.00 -> 21.5 mm
- net CV_OUT: track 0.00 -> 18.0 mm
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- added copper zone on B.Cu, net GND
- added copper zone on F.Cu, net GND
Other:
- outline, holes or cut-outs redrawn
