File: KiCAD/MixtapeNEO-3000.sch (KiCad schematic (older format))
At the start: 54 parts, among them J1 CONN_01X04, J18 Con_3-5V, J2 CONN_01X04, J3 CONN_02X03, J5 CONN_01X02_MALE, J7 USB_OTG, SW1 SW_Push, SW2 SW_Push, SW3 SW_Push, SW6 SW_Push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

Commit message: adding schematic
Other:
- moved on the sheet: C5, C6, C7, J1, R14, R15, Speaker1, U2, board1

Commit message: all footprints done
Parts:
- removed C7: 10uF, 8BitMixtape-3000:C_1206_HandSoldering, symbol C
- added C7: 220uF, 8BitMixtape-3000:C_1206_HandSoldering, symbol CP
- BT1, BT2: footprint (none) -> 8BitMixtape-3000:BAT_Holder_AAA-new
- POT1-MAIN1, POT2-CV1: footprint 8BitMixtape-3000:Poti_Mouser -> 8BitMixtape-3000:Potentiometer_backPads_noHole
- POT3-Vol1: footprint 8Bit_ESPTINY86-Mixtape:Potentiometer_wheel -> 8BitMixtape-3000:Potentiometer_wheel
- SW1: footprint 8Bit-MOJ-MIKRO-Kaseta:Push_SWITCH_hole -> 8BitMixtape-3000:Push_SWITCH_hole
- SW4: renamed from SW6; footprint 8Bit-MOJ-MIKRO-Kaseta:SW_SPST_FSMSM -> 8BitMixtape-3000:SW_SPST_FSMSM
- renumbered C6 to C5, C5 to C6, J18 to J4, J7 to J5, J5 to J6
Connections:
- net GND: now also C7.2
- net VCC: now also C7.1
Changed lines of the file:
@@
 F 0 "POT2-CV1" V 5025 6150 50  0000 C CNN
 F 1 "POT 10K lin" V 5100 6150 50  0000 C CNN
-F 2 "8BitMixtape-3000:Poti_Mouser" H 5200 6150 50  0001 C CNN
+F 2 "8BitMixtape-3000:Potentiometer_backPads_noHole" H 5200 6150 50  0001 C CNN
 F 3 "" H 5200 6150 50  0001 C CNN
 	1    5200 6150
@@
 F 0 "POT1-MAIN1" V 5025 3950 50  0000 C CNN
 F 1 "POT 10K lin" V 5100 3950 50  0000 C CNN
-F 2 "8BitMixtape-3000:Poti_Mouser" H 5200 3950 50  0001 C CNN
+F 2 "8BitMixtape-3000:Potentiometer_backPads_noHole" H 5200 3950 50  0001 C CNN
 F 3 "" H 5200 3950 50  0001 C CNN
 	1    5200 3950
@@
 F 0 "POT3-Vol1" V 7575 3800 50  0000 C CNN
 F 1 "POT 10k" V 7650 3800 50  0000 C CNN
-F 2 "8Bit_ESPTINY86-Mixtape:Potentiometer_wheel" H 7750 3800 50  0001 C CNN
+F 2 "8BitMixtape-3000:Potentiometer_wheel" H 7750 3800 50  0001 C CNN
 F 3 "" H 7750 3800 50  0001 C CNN
 	1    7750 3800
@@
 CV_OUT
 $Comp
-L CONN_01X02_MALE J5
+L CONN_01X02_MALE J6
 U 1 1 5B474264
 P 6800 5700
-F 0 "J5" H 6800 5875 50  0000 C CNN
+F 0 "J6" H 6800 5875 50  0000 C CNN
 F 1 "CONN_01X02_MALE" H 6800 5500 50  0000 C CNN
 F 2 "Resistors_SMD:R_0612" H 6800 5800 50  0001 C CNN
@@
 F 0 "SW1" H 2550 1100 50  0000 L CNN
 F 1 "SW_Push" H 2500 940 50  0000 C CNN
-F 2 "8Bit-MOJ-MIKRO-Kaseta:Push_SWITCH_hole" H 2500 1200 50  0001 C CNN
+F 2 "8BitMixtape-3000:Push_SWITCH_hole" H 2500 1200 50  0001 C CNN
 F 3 "" H 2500 1200 50  0001 C CNN
 	1    2500 1000
@@
 $EndComp
 $Comp
-L USB_OTG J7
+L USB_OTG J5
 U 1 1 5B4A98DA
 P 1950 1750
-F 0 "J7" H 1750 2200 50  0000 L CNN
+F 0 "J5" H 1950 2200 50  0000 L CNN
 F 1 "USB_OTG" H 1750 2100 50  0000 L CNN
 F 2 "8BitMixtape-3000:USB_Micro-B" H 2100 1700 50  0001 C CNN
@@
 $EndComp
 $Comp
-L SW_Push SW6
+L SW_Push SW4
 U 1 1 5B4ADF33
 P 6600 6100
-F 0 "SW6" H 6650 6200 50  0000 L CNN
+F 0 "SW4" H 6650 6200 50  0000 L CNN
 F 1 "SW_Push" H 6600 6040 50  0000 C CNN
-F 2 "8Bit-MOJ-MIKRO-Kaseta:SW_SPST_FSMSM" H 6600 6300 50  0001 C CNN
+F 2 "8BitMixtape-3000:SW_SPST_FSMSM" H 6600 6300 50  0001 C CNN
 F 3 "" H 6600 6300 50  0001 C CNN
 	1    6600 6100
@@
 	5850 3950 6100 3950
 Wire Wire Line
-	6100 3950 6100 4250
-Wire Wire Line
-	6100 4250 6100 4650
+	6100 3950 6100 4650
 Wire Wire Line
 	6100 4650 6400 4650
@@
 	6100 6150 5800 6150
 Wire Wire Line
-	6100 4850 6100 5100
-Wire Wire Line
-	6100 5100 6100 6150
+	6100 4850 6100 6150
 Wire Wire Line
 	6100 4850 6400 4850
 Wire Wire Line
-	3100 4750 3350 4750
-Wire Wire Line
-	3350 4750 3800 4750
-Wire Wire Line
-	3800 4750 4400 4750
-Wire Wire Line
-	4400 4750 4800 4750
-Wire Wire Line
-	4800 4750 6400 4750
-Wire Wire Line
-	3350 4500 3350 4750
-Wire Wire Line
-	3350 4750 3350 4950
+	3100 4750 6400 4750
+Wire Wire Line
+	3350 4500 3350 4950
 Connection ~ 3350 4750
 Wire Wire Line
@@
 	3350 5250 3350 5450
 Wire Wire Line
-	5200 5800 5200 5900
-Wire Wire Line
-	5200 5900 5200 6000
+	5200 5800 5200 6000
 Wire Wire Line
 	5200 6300 5200 6500
@@
 Connection ~ 3800 4750
 Wire Wire Line
-	4300 5100 4400 5100
-Wire Wire Line
-	4400 5100 4500 5100
+	4300 5100 4500 5100
 Wire Wire Line
 	4400 5100 4400 4750
@@
 	4300 5600 4300 5800
 Wire Wire Line
-	4300 5800 4400 5800
-Wire Wire Line
-	4400 5800 4500 5800
-Wire Wire Line
-	4500 5800 4500 5750
-Wire Wire Line
-	4500 5750 4500 5600
+	4300 5800 4500 5800
+Wire Wire Line
+	4500 5800 4500 5600
 Connection ~ 4400 5800
 Wire Wire Line
 	6250 4550 6400 4550
 Wire Wire Line
-	6250 3000 6250 3300
-Wire Wire Line
-	6250 3300 6250 3550
-Wire Wire Line
-	6250 3550 6250 4550
+	6250 3000 6250 4550
 Wire Wire Line
 	6250 3550 6550 3550
@@
 	9100 3750 9100 3950
 Wire Wire Line
-	2150 4750 2500 4750
-Wire Wire Line
-	2500 4750 2800 4750
+	2150 4750 2800 4750
 Wire Wire Line
 	2150 4350 2250 4350
@@
 	6900 5400 7300 5400
 Wire Wire Line
-	9100 4450 9300 4450
-Wire Wire Line
-	9300 4450 9650 4450
+	9100 4450 9650 4450
 Wire Wire Line
 	9300 4450 9300 4550
 Wire Wire Line
-	9650 4300 9650 4450
-Wire Wire Line
-	9650 4450 9650 4550
+	9650 4300 9650 4550
 Connection ~ 9300 4450
 Wire Wire Line
-	9100 4950 9300 4950
-Wire Wire Line
-	9300 4950 9650 4950
+	9100 4950 9650 4950
 Wire Wire Line
 	9300 4950 9300 4850
 Wire Wire Line
-	9650 4850 9650 4950
-Wire Wire Line
-	9650 4950 9650 5150
+	9650 4850 9650 5150
 Connection ~ 9300 4950
 Connection ~ 9650 4450
@@
 Connection ~ 6400 5400
 Wire Wire Line
-	6850 3550 7300 3550
-Wire Wire Line
-	7300 3550 7750 3550
+	6850 3550 7750 3550
 Wire Wire Line
 	7750 3550 7750 3650
 Wire Wire Line
-	7900 3800 8100 3800
-Wire Wire Line
-	8100 3800 8400 3800
+	7900 3800 8400 3800
 Wire Wire Line
 	8400 3800 8400 3550
@@
 	3800 5850 3900 5850
 Wire Wire Line
-	3800 5600 3800 5750
-Wire Wire Line
-	3800 5750 3800 5850
+	3800 5600 3800 5850
 Wire Wire Line
 	850  5950 1450 5950
@@
 	7300 3100 7550 3100
 Wire Wire Line
-	7300 3100 7300 3550
-Wire Wire Line
-	7300 3550 7300 3650
+	7300 3100 7300 3650
 Wire Wire Line
 	5950 3000 5950 3200
@@
 	1400 1450 1400 1500
 Wire Wire Line
-	1800 1150 2300 1150
-Wire Wire Line
-	2300 1150 2750 1150
-Wire Wire Line
-	2750 1150 3200 1150
-Wire Wire Line
-	3200 1150 3600 1150
+	1800 1150 3600 1150
 Wire Wire Line
 	3600 1150 3600 900
@@
 	6600 6300 6400 6300
 Wire Wire Line
-	6400 4950 6400 5400
-Wire Wire Line
-	6400 5400 6400 5900
+	6400 4950 6400 5900
 Wire Wire Line
 	6400 6300 6400 6500
@@
 	4200 2750 11150 2750
 $Comp
-L CONN_01X02 J18
+L CONN_01X02 J4
 U 1 1 5B4D3718
 P 2600 2000
-F 0 "J18" H 2600 2150 50  0000 C CNN
+F 0 "J4" H 2600 2150 50  0000 C CNN
 F 1 "Con_3-5V" V 2700 2000 50  0000 C CNN
 F 2 "8BitMixtape-3000:Bat_connector" H 2600 2000 50  0001 C CNN
@@
 $EndComp
 $Comp
-L C C6
+L C C5
 U 1 1 5C5FEF8C
 P 7000 1500
-F 0 "C6" H 7025 1600 50  0000 L CNN
+F 0 "C5" H 7025 1600 50  0000 L CNN
 F 1 "10uF" H 7025 1400 50  0000 L CNN
 F 2 "8BitMixtape-3000:C_1206_HandSoldering" H 7038 1350 50  0001 C CNN
@@
 $EndComp
 $Comp
-L C C5
+L C C6
 U 1 1 5C5FEF8D
 P 7750 2200
-F 0 "C5" H 7775 2300 50  0000 L CNN
+F 0 "C6" H 7775 2300 50  0000 L CNN
 F 1 "1uF" H 7775 2100 50  0000 L CNN
 F 2 "8BitMixtape-3000:C_1206_HandSoldering" H 7788 2050 50  0001 C CNN
@@
 $EndComp
 Wire Wire Line
-	7750 1500 7850 1500
-Wire Wire Line
-	7850 1500 8000 1500
+	7750 1500 8000 1500
 Wire Wire Line
 	7450 1500 7150 1500
@@
 	9150 1150 9150 1600
 Wire Wire Line
-	9000 1600 9150 1600
-Wire Wire Line
-	9150 1600 9300 1600
+	9000 1600 9300 1600
 $Comp
 L VCC #PWR030
@@
 	8000 1650 7750 1650
 Wire Wire Line
-	7750 1650 7750 1800
-Wire Wire Line
-	7750 1800 7750 2050
+	7750 1650 7750 2050
 Wire Wire Line
 	8000 1800 7750 1800
@@
 	1    0    0    -1
 $EndComp
-$Comp
-L C C7
-U 1 1 5C5FEF97
-P 5750 1150
-F 0 "C7" H 5775 1250 50  0000 L CNN
-F 1 "10uF" H 5775 1050 50  0000 L CNN
-F 2 "8BitMixtape-3000:C_1206_HandSoldering" H 5788 1000 50  0001 C CNN
-F 3 "" H 5750 1150 50  0001 C CNN
-	1    5750 1150
-	-1   0    0    1
-$EndComp
 Wire Wire Line
 	5750 1300 5750 1400
@@
 F 0 "BT1" H 900 2000 50  0000 L CNN
 F 1 "Battery_Cell" H 900 1900 50  0000 L CNN
-F 2 "" V 800 1960 50  0001 C CNN
+F 2 "8BitMixtape-3000:BAT_Holder_AAA-new" V 800 1960 50  0001 C CNN
 F 3 "" V 800 1960 50  0001 C CNN
 	1    800  1900
@@
 F 0 "BT2" H 900 2400 50  0000 L CNN
 F 1 "Battery_Cell" H 900 2300 50  0000 L CNN
-F 2 "" V 800 2360 50  0001 C CNN
+F 2 "8BitMixtape-3000:BAT_Holder_AAA-new" V 800 2360 50  0001 C CNN
 F 3 "" V 800 2360 50  0001 C CNN
 	1    800  2300
@@
 Wire Notes Line
 	4150 2750 550  2750
+$Comp
+L CP C7
+U 1 1 5C602B8D
+P 5750 1150
+F 0 "C7" H 5775 1250 50  0000 L CNN
+F 1 "220uF" H 5775 1050 50  0000 L CNN
+F 2 "8BitMixtape-3000:C_1206_HandSoldering" H 5788 1000 50  0001 C CNN
+F 3 "" H 5750 1150 50  0001 C CNN
+	1    5750 1150
+	1    0    0    -1
+$EndComp
 $EndSCHEMATC

Commit message: complete revision
Parts:
- added R99: 0, 8BitMixtape-3000-clean:R_1206_HandSoldering, symbol R
- BT1, BT2: footprint 8BitMixtape-3000:BAT_Holder_AAA-new -> 8BitMixtape-3000-clean:BAT_Holder_AAA-new_noHole
- C1, C2, C3, C4, C5, C6, C7: footprint 8BitMixtape-3000:C_1206_HandSoldering -> 8BitMixtape-3000-clean:C_1206_HandSoldering
- D-OUT1, D-POW1: footprint 8BitMixtape-3000:LED_2835_minimal -> 8BitMixtape-3000-clean:LED_2835_minimal
- J1, J2: footprint 8BitMixtape-3000:Angled_1x04_Pitch2.54mm-flip -> 8BitMixtape-3000-clean:Angled_1x04_Pitch2.54mm-flip
- J3: footprint 8BitMixtape-3000:Socket_Strip_Straight_2x03_Pitch2.54mm -> 8BitMixtape-3000-clean:Socket_Strip_Straight_2x03_Pitch2.54mm
- J4: footprint 8BitMixtape-3000:Bat_connector -> 8BitMixtape-3000-clean:Bat_connector_SMD
- J5: footprint 8BitMixtape-3000:USB_Micro-B -> 8BitMixtape-3000-clean:USB_Micro-B
- J6: footprint Resistors_SMD:R_0612 -> 8BitMixtape-3000-clean:R_0612
- Jack1, Jack2: footprint 8BitMixtape-3000:AUDIO-Jack_3.5mm_5Pin -> 8BitMixtape-3000-clean:AUDIO-Jack_3.5mm_5Pin
- NEO1, NEO2, NEO3, NEO4, NEO5, NEO6, NEO7, NEO8: footprint 8BitMixtape-3000:Mixtape_NEO_WS2812B -> 8BitMixtape-3000-clean:Mixtape_NEO_WS2812B
- POT1-MAIN1, POT2-CV1: footprint 8BitMixtape-3000:Potentiometer_backPads_noHole -> 8BitMixtape-3000-clean:Potentiometer_backPads_noHole
- POT3-Vol1: footprint 8BitMixtape-3000:Potentiometer_wheel -> 8BitMixtape-3000-clean:Potentiometer_wheel
- R1, R10, R11, R12, R13, R14, R15, R2, R3, R4, R5, R6, R7, R8, R9: footprint 8BitMixtape-3000:R_1206_HandSoldering -> 8BitMixtape-3000-clean:R_1206_HandSoldering
- SW1: footprint 8BitMixtape-3000:Push_SWITCH_hole -> 8BitMixtape-3000-clean:Push_SWITCH_hole
- SW2, SW3: footprint 8BitMixtape-3000:SW_PUSH-12mm_3D -> 8BitMixtape-3000-clean:TACTILE-PTH_6mm_SMD
- SW4: footprint 8BitMixtape-3000:SW_SPST_FSMSM -> 8BitMixtape-3000-clean:SW_SPST_FSMSM
- Speaker1: footprint 8BitMixtape-3000:Socket_Strip_Straight_1x02_Pitch2.54mm -> 8BitMixtape-3000-clean:SpeakerPads_SMD
- U1: footprint 8BitMixtape-3000:Attiny_DIP-8_W7.62mm -> 8BitMixtape-3000-clean:Attiny_DIP-8_W7.62mm_mod
- U2: footprint Housings_SOIC:SO-8_5.3x6.2mm_Pitch1.27mm -> 8BitMixtape-3000-clean:SO-8_5.3x6.2mm_Pitch1.27mm
- U3: footprint TO_SOT_Packages_SMD:TO-252-3_TabPin2 -> 8BitMixtape-3000-clean:TO-252-3_TabPin2
- board1: footprint 8BitMixtape-3000:MixtapeNEO-3000 -> 8BitMixtape-3000-clean:MixtapeNEO-3000
Connections:
- net Sound_IN is gone; now on net CV_IN: POT2-CV1.1, R10.2
- net CV_IN: now also R99.1; no longer Jack1.2 (T)
- net PB1: now also J2.3 (P3)
- net Sound_OUT: now also Jack2.5 (TN); no longer J2.3 (P3), Jack2.2 (T), POT3-Vol1.2
- new net: Jack2.2 (T), POT3-Vol1.2
- new net: Jack1.2 (T), R99.2
